File: eagle/TouScruino-v3.sch (EAGLE design)
At the start: 42 parts, among them J1 AVR_ISP, Q1 8MHz, Q2 MMBT2222A, Q3 8MHz, U1 ATMEGA1284P, U2 PJ28004C, U3 ARDUINO_SHIELD, U4 MCP73831, U5 MIC5209-3.3YS, X1 USBSMD

Commit message: 
Parts:
- removed C3: 0.1uF, SparkFun:CAP0805
- removed D1: BAT54C, wibauxl:BAT54C
- removed J1: AVR_ISP, SparkFun:AVR_SPI_PRG_6PTH
- removed SJ2: SJ_2WAYS_1-2, wibauxl:SJ_2WAYS_1-2
- added C11: 18pF, SparkFun:CAP0603-CAP
- added Q4: 8MHz, wibauxl:CRYSTAL_5X3.2
- added S2: SWITCH-MOMENTARY-2SMD, SparkFun:SWITCH-MOMENTARY-2SMD
- added U$4: AR1020, wibauxl:AR1020
- added U$6: ATSAM3S_C, wibauxl:ATSAM3S_C
- C2: value 0.1uF -> 18pF; device SparkFun:CAP0805 -> SparkFun:CAP0603-CAP
- JP1: value (none) -> M20; device SparkFun:ARDUINO_SERIAL_PROGRAMPTH -> SparkFun:M20
- R2: value 10K -> 10k
- R4: value 75K -> 20k
- U1: value ATMEGA1284P -> uSD-SOCKET; device wibauxl:ATMEGA324A -> SparkFun:USD-SOCKETNEW
Connections:
- removed net A0/D24: U1.(PCINT0/ADC0)PA0, U3.A0
- removed net A1/D25: U1.(PCINT1/ADC1)PA1, U3.A1
- removed net A2/D26: U1.(PCINT2/ADC2)PA2, U3.A2
- removed net A3/D27: U1.(PCINT3/ADC3)PA3, U3.A3
- removed net A4/D28: U1.(PCINT4/ADC4)PA4, U3.A4
- removed net A5/D29: U1.(PCINT5/ADC5)PA5, U3.A5
- removed net A6/D30: U1.(PCINT6/ADC6)PA6, U2.X-
- removed net A7/D31: U1.(PCINT7/ADC7)PA7, U2.Y+
- removed net AREF: C1.2, U1.AREF
- removed net D0/RX: JP1.TXO, U1.(PCINT24/RXD0)PD0, U3.RX
- removed net D1/TX: JP1.RXI, U1.(PCINT25/TXD0)PD1, U3.TX
- removed net D10/PWM4: U1.(PCINT31/OC2A)PD7, U3.D10
- removed net D11/MOSI: J1.4, U1.(PCINT13/MOSI)PB5, U2.DB5, U3.D11
- removed net D12/MISO: J1.1, U1.(PCINT14/MISO)PB6, U2.DB6, U3.D12
- removed net D13/SCK: J1.3, R5.2, U1.(PCINT15/SCK)PB7, U2.DB7, U3.D13
- removed net D14: U1.(PCINT8/XCK0/T0)PB0, U2.DB0, U2.Y-
- removed net D15: U1.(PCINT9/CLKO/T1)PB1, U2.DB1, U2.X+
- removed net D16: U1.(PCINT10/INT2/AIN0)PB2, U2.DB2
- removed net D17: U1.(PCINT11/OC0A/AIN1)PB3, U2.DB3
- removed net D18: U1.(PCINT12/OC0B/!SS!)PB4, U2.DB4
- removed net D19/SCL: JP3.1, U1.(PCINT16/SCL)PC0
- removed net D2/RX1: U1.(PCINT26/INT0/RXD1)PD2, U3.D2
- removed net D20/SDA: JP3.2, U1.(PCINT17/SDA)PC1
- removed net D21: U1.(PCINT21/TDI)PC5, U2.DC
- removed net D22: D1.A2, U1.(PCINT22/TOSC1)PC6, U2.WR
- removed net D23: D1.A1, U1.(PCINT23/TOSC2)PC7, U2.RD
- removed net D3/TX1: U1.(PCINT27/INT1/TXD1)PD3, U3.D3
- removed net D6/PWM2: U1.(PCINT29/OC1A)PD5, U3.D6
- removed net D8: U1.(PCINT20/TDO)PC4, U3.D8
- removed net D9/PWM3: U1.(PCINT30/OC2B/ICP)PD6, U3.D9
- removed net DTR: C2.2, JP1.DTR
- removed net LCD_RES: SJ2.2, U2.RES
- new net A.A0: U$6.PA17/AD0, U3.A0
- new net A.A1: U$6.PB0/AD4, U3.A1
- new net A.A2: U$6.PB1/AD5, U3.A2
- new net A.A3: U$6.PB2/AD6, U3.A3
- new net A.A4: U$6.PB3/AD7, U3.A4
- new net A.A5: U$6.PC12/NCS3/AD12, U3.A5
- new net A.AREF: U$6.ADVREF, U3.AREF
- new net A.D0/RX0: U$6.PA21/RXD1/AD8, U3.RX
- new net A.D1/TX0: U$6.PA22/TXD1/AD9, U3.TX
- new net A.D10: U$6.PA11/NPCS0, U3.D10
- new net A.D11/MISO: U$4.SDO/IRQ, U$6.PA12/MISO, U3.D11
- new net A.D12/MOSI: U$4.SDI/SDA, U$6.PA13/MOSI, U3.D12
- new net A.D13: U3.D13
- new net A.D13/SCK: R5.2, U$4.SCK/SCL, U$6.PA14/SCK
- new net A.D2/RX1: U$6.PA9/URXD0, U3.D2
- new net A.D3/TX1: U$6.PA10/UTXD0, U3.D3
- new net A.D4: U$6.PA24/A20, U3.D4
- new net A.D5: U$6.PC13/AD10, U3.D5
- new net A.D6: U$6.PA15/TIOA1, U3.D6
- new net A.D7/DAC0: U$6.PB13/DAC0, U3.D7
- new net A.D8/DAC1: U$6.PB14/DAC1, U3.D8
- new net A.D9: U$6.PA16/TIOB1, U3.D9
- new net A.SCL: JP3.1, U$6.PA4/SCL0
- new net A.SDA: JP3.2, U$6.PA3/SDA0
- new net A0: U$6.PC18/A0
- new net A1: U$6.PC19/A1, U2.DC
- new net A10: U$6.PC28/A10
- new net A11: U$6.PC29/A11
- new net A12: U$6.PC30/A12
- new net A13: U$6.PC31/A13
- new net A14: U$6.PA18/A14/AD1
- new net A15: U$6.PA19/A15/AD2
- new net A16: U$6.PA20/A16/AD3
- new net A17: U$6.PA0/A17
- new net A18: U$6.PA1/A18
- new net A19: U$6.PA23/A19
- new net A2: U$6.PC20/A2
- new net A21: U$6.PC16/A21
- new net A22: U$6.PC17/A22
- new net A3: U$6.PC21/A3
- new net A4: U$6.PC22/A4
- new net A5: U$6.PC23/A5
- new net A6: U$6.PC24/A6
- new net A7: U$6.PC25/A7
- new net A8: U$6.PC26/A8
- new net A9: U$6.PC27/A9
- new net D0: U$6.PC0/D0, U2.DB0
- new net D1: U$6.PC1/D1, U2.DB1
- new net D2: U$6.PC2/D2, U2.DB2
- new net D3: U$6.PC3/D3, U2.DB3
- new net D5: U$6.PC5/D5, U2.DB5
- new net D6: U$6.PC6/D6, U2.DB6
- new net LCD.BL: U$6.PA2/PWMH2
- new net LCD_CS: U$6.PC15/NCS1/AD11, U2.CS
- new net N$10: U$6.VDDCORE@1, U$6.VDDCORE@2, U$6.VDDCORE@3, U$6.VDDCORE@4, U$6.VDDOUT, U$6.VDDPLL
- new net N$11: R4.2, U$4.WAKE
- new net N$14: S2.2, U$6.ERASE/PB12
- new net N$45: C2.1, Q4.1, U$6.PA7/XIN32
- new net N$46: C11.1, Q4.2, U$6.PA8/XOUT32
- new net PD_CS: U$6.PC14/NCS0
- new net RD: U$6.PC11/NRD, U2.RD
- new net SD.CD: U$6.PA25/A23, U1.SHIELD@2
- new net SD.CLK: U$6.PA29/MCCCK, U1.SCK
- new net SD.CMD: U$6.PA28/MCCDA, U1.DI
- new net SD.D0: U$6.PA30/MCDA0, U1.DO
- new net SD.D1: U$6.PA31/MCDA1, U1.RSV
- new net SD.D2: U$6.PA26/MCDA2, U1.NC
- new net SD.D3: U$6.PA27/MCDA3, U1.CS
- new net TCK: U$6.TCK/PB7
- new net TDI: U$6.TDI/PB4
- new net TDO: U$6.TDO/PB5
- new net TMS: U$6.TMS/PB6
- new net TS.CS: U$4.SS, U$6.PA5/NPCS3
- new net TS.IRQ: U$4.SIQ, U$6.PA6
- new net USB.D+: U$6.DDP/PB11, X1.D+
- new net USB.D-: U$6.DDM/PB10, X1.D-
- new net WR: U$6.PC8/NWE, U2.WR
- new net X+: U$4.X+, U2.X+
- new net X-: U$4.X-, U2.X-
- new net Y+: U$4.Y+, U2.Y+
- new net Y-: R4.1, U$4.Y-, U2.Y-
- net 3.3V: now also C1.2, S2.1, U$4.M1, U$4.VDD, U$6.VDDIN, U$6.VDDIO@1, U$6.VDDIO@2, U$6.VDDIO@3, U$6.VDDIO@4, U$6.VDDIO@5; no longer C3.2, J1.2, JP1.VCC, U1.AVCC, U1.VCC@1, U1.VCC@2
- net D4: now also U$6.PC4/D4, U2.DB4; no longer U1.(PCINT18/TCK)PC2, U3.D4
- net D5/PWM1: no longer U1.(PCINT28/OC1B)PD4, U3.D5
- net D7: now also U$6.PC7/D7, U2.DB7; no longer U1.(PCINT19/TMS)PC3, U3.D7
- net GND: now also C11.2, C2.2, S1.1, U$4.M2, U$4.SX+, U$4.SX-, U$4.SY+, U$4.SY-, U$4.VSS, U$6.GND@1, U$6.GND@2, U$6.GND@3, U$6.GND@4, U$6.GND@5, U$6.JTAGSEL, U$6.TST, U1.SHIELD@1, U1.SHIELD@3; no longer C3.1, J1.6, JP1.CTS, JP1.GND, R4.1, S1.2, U1.GND@1, U1.GND@2, U1.GND@3, U2.CS
- net N$1: now also U$6.XIN/PB9; no longer U1.XTAL1
- net N$2: now also U$6.XOUT/PB8; no longer U1.XTAL2
- net N$9: now also R2.1, S1.2, U$6.NRST; no longer D1.K, R4.2, SJ2.1
- net RES: no longer C2.1, J1.5, R2.1, S1.1, SJ2.3, U1.RESET
- net VUSB: now also JP5.3
Other:
- note removed: "For the touchscreen to work"
- note removed: "analogReference needs to be set to DEFAULT: 3.3V"
- note removed: "so AREF is left intentionaly unconnected on the shield"
- moved on the sheet: C1, C10, C2, C9, JP4, LED2, Q1, Q2, Q3, R2, R4, R5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
